File: PCB/Eagle/V3/Espressomaschine.brd (EAGLE design)
At the start: 73.6 x 63.6 mm, 82 parts, among them IC1 NE555D, IC5 MCP23017SO, Q1 IRLML5203, U1 BSS138BK_SOT_23, U2 BSS138BK_SOT_23, U3 BSS138BK_SOT_23, U4 BSS138BK_SOT_23, U5 ADS1115IDGST, U6 BSS138BK_SOT_23

Commit message: Finalized PCB V3
Parts:
- added R19: 10k, rcl:R0603
- moved Q1 1.80 mm to (79.2, 59.2)
Connections:
- net +3V3: now also R19.2
- net ADS_RDY: now also R19.1
Routing:
- net +5V: track 231.5 -> 242.0 mm
- net 230V_N: track 7.42 -> 15.4 mm
- net 230V_L: track 7.42 -> 14.8 mm
- net N$52: track 0.00 -> 2.54 mm
- net N$24: track 5.98 -> 7.78 mm
- net DISP_LED: track 7.39 -> 5.59 mm
- net +3V3: track 269.9 -> 270.9 mm, vias 12 -> 13
- net ADS_RDY: track 10.1 -> 11.0 mm
- net DISP_SDO: track 44.0 -> 44.7 mm
Other:
- board text added: "BU heater"
- board text added: "BU valve"
- board text added: "CS"
- board text added: "DC"
- board text added: "LED"
- board text added: "SCK"
- board text added: "SDI"
- board text added: "SDO"
- board text added: "boiler valve"
- board text added: "reset"
