File: PCB/Eagle/V3/Espressomaschine.sch (EAGLE design)
At the start: 82 parts, among them IC1 NE555D, IC5 MCP23017SO, Q1 IRLML5203, U1 BSS138BK_SOT_23, U2 BSS138BK_SOT_23, U3 BSS138BK_SOT_23, U4 BSS138BK_SOT_23, U5 ADS1115IDGST, U6 BSS138BK_SOT_23

Commit message: Finalized PCB V3
Parts:
- added R19: 10k, rcl:R-EU_R0603
Connections:
- net +3V3: now also R19.2
- net ADS_RDY: now also R19.1
Changed lines of the file:
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@@
 <part name="U$13" library="PINHD_eigen" deviceset="PINHD-1X1" device="SMD_RM1.27"/>
 <part name="U$14" library="PINHD_eigen" deviceset="PINHD-1X1" device="SMD_RM1.27"/>
+<part name="R19" library="rcl" library_urn="urn:adsk.eagle:library:334" deviceset="R-EU_" device="R0603" package3d_urn="urn:adsk.eagle:package:23555/3" value="10k"/>
 </parts>
 <sheets>
@@
 <instance part="U$13" gate="G$1" x="-91.44" y="15.24" smashed="yes" rot="R180"/>
 <instance part="U$14" gate="G$1" x="-91.44" y="10.16" smashed="yes" rot="R180"/>
+<instance part="R19" gate="G$1" x="27.94" y="40.64" smashed="yes" rot="R90">
+<attribute name="NAME" x="26.4414" y="36.83" size="1.778" layer="95" rot="R90"/>
+<attribute name="VALUE" x="31.242" y="36.83" size="1.778" layer="96" rot="R90"/>
+</instance>
 </instances>
 <busses>
@@
 <pinref part="+3V1" gate="G$1" pin="+3V3"/>
 <wire x1="20.32" y1="48.26" x2="20.32" y2="50.8" width="0.1524" layer="91"/>
+<pinref part="R19" gate="G$1" pin="2"/>
+<wire x1="20.32" y1="48.26" x2="27.94" y2="48.26" width="0.1524" layer="91"/>
+<wire x1="27.94" y1="48.26" x2="27.94" y2="45.72" width="0.1524" layer="91"/>
 </segment>
 <segment>
@@
 <label x="-83.82" y="2.54" size="1.778" layer="95"/>
 </segment>
-</net>
+<segment>
+<pinref part="R19" gate="G$1" pin="1"/>
+<wire x1="27.94" y1="35.56" x2="27.94" y2="30.48" width="0.1524" layer="91"/>
+<label x="27.94" y="25.4" size="1.778" layer="95" rot="R90"/>
+</segment>
+</net>
